Commit message: - noluyo amk

File: models/rotors_description/urdf/component_snippets.xacro (robot description, xacro)
@@ -118,5 +118,5 @@
     </gazebo>
   </xacro:macro>
-  <!-- Macro to add the gps_plugin. -->
+    <!-- Macro to add the gps_plugin. -->
   <xacro:macro name="gps_plugin_macro" params="namespace gps_noise">
     <gazebo>
@@ -127,29 +127,6 @@
     </gazebo>
   </xacro:macro>
-  <!-- Macro to add the magnetometer_plugin. -->
-  <xacro:macro name="magnetometer_plugin_macro" params="namespace pub_rate noise_density random_walk bias_correlation_time mag_topic">
-    <gazebo>
-      <plugin name="magnetometer_plugin" filename="libgazebo_magnetometer_plugin.so">
-        <robotNamespace>${namespace}</robotNamespace>
-        <pubRate>${pub_rate}</pubRate>
-        <noiseDensity>${noise_density}</noiseDensity>
-        <randomWalk>${random_walk}</randomWalk>
-        <biasCorrelationTime>${bias_correlation_time}</biasCorrelationTime>
-        <magTopic>${mag_topic}</magTopic>
-      </plugin>
-    </gazebo>
-  </xacro:macro>
-  <!-- Macro to add the barometer_plugin. -->
-  <xacro:macro name="barometer_plugin_macro" params="namespace pub_rate baro_topic">
-    <gazebo>
-      <plugin name="barometer_plugin" filename="libgazebo_barometer_plugin.so">
-        <robotNamespace>${namespace}</robotNamespace>
-        <pubRate>${pub_rate}</pubRate>
-        <baroTopic>${baro_topic}</baroTopic>
-      </plugin>
-    </gazebo>
-  </xacro:macro>
   <!-- Macro to add the mavlink interface. -->
-  <xacro:macro name="mavlink_interface_macro" params="namespace imu_sub_topic gps_sub_topic mag_sub_topic baro_sub_topic mavlink_addr mavlink_udp_port mavlink_tcp_port serial_enabled serial_device baudrate qgc_addr qgc_udp_port sdk_addr sdk_udp_port hil_mode hil_state_level vehicle_is_tailsitter send_vision_estimation send_odometry enable_lockstep use_tcp">
+  <xacro:macro name="mavlink_interface_macro" params="namespace imu_sub_topic gps_sub_topic mavlink_addr mavlink_udp_port serial_enabled serial_device baudrate qgc_addr qgc_udp_port hil_mode hil_state_level vehicle_is_tailsitter">
     <gazebo>
       <plugin name="mavlink_interface" filename="libgazebo_mavlink_interface.so">
@@ -157,9 +134,6 @@
         <imuSubTopic>${imu_sub_topic}</imuSubTopic>
         <gpsSubTopic>${gps_sub_topic}</gpsSubTopic>
-        <magSubTopic>${mag_sub_topic}</magSubTopic>
-        <baroSubTopic>${baro_sub_topic}</baroSubTopic>
         <mavlink_addr>$(arg mavlink_addr)</mavlink_addr>
         <mavlink_udp_port>$(arg mavlink_udp_port)</mavlink_udp_port>
-        <mavlink_tcp_port>$(arg mavlink_tcp_port)</mavlink_tcp_port>
         <serialEnabled>$(arg serial_enabled)</serialEnabled>
         <serialDevice>$(arg serial_device)</serialDevice>
@@ -167,13 +141,7 @@
         <qgc_addr>$(arg qgc_addr)</qgc_addr>
         <qgc_udp_port>$(arg qgc_udp_port)</qgc_udp_port>
-        <sdk_addr>$(arg sdk_addr)</sdk_addr>
-        <sdk_udp_port>$(arg sdk_udp_port)</sdk_udp_port>
         <hil_mode>$(arg hil_mode)</hil_mode>
         <hil_state_level>$(arg hil_state_level)</hil_state_level>
         <vehicle_is_tailsitter>$(arg vehicle_is_tailsitter)</vehicle_is_tailsitter>
-        <send_vision_estimation>$(arg send_vision_estimation)</send_vision_estimation>
-        <send_odometry>$(arg send_odometry)</send_odometry>
-        <enable_lockstep>$(arg enable_lockstep)</enable_lockstep>
-        <use_tcp>$(arg use_tcp)</use_tcp>
         <motorSpeedCommandPubTopic>/gazebo/command/motor_speed</motorSpeedCommandPubTopic>
         <control_channels>

File: models/rotors_description/urdf/iris.xacro (robot description, xacro)
@@ -30,9 +30,5 @@
   <!-- Property Blocks -->
   <xacro:property name="body_inertia">
-    <inertia
-    ixx="${1/12 * mass * (body_height * body_height + body_width * body_width)}"
-    iyy="${1/12 * mass * (body_height * body_height + body_width * body_width)}"
-    izz="${1/12 * mass * (body_width * body_width + body_width * body_width)}"
-    ixy="0.0" ixz="0.0" iyz="0.0" /> <!-- [kg.m^2] [kg.m^2] [kg.m^2] [kg.m^2] [kg.m^2] [kg.m^2] -->
+    <inertia ixx="0.0347563" ixy="0.0" ixz="0.0" iyy="0.0458929" iyz="0.0" izz="0.0977" /> <!-- [kg.m^2] [kg.m^2] [kg.m^2] [kg.m^2] [kg.m^2] [kg.m^2] -->
   </xacro:property>
   <!-- inertia of a single rotor, assuming it is a cuboid. Height=3mm, width=15mm -->

File: models/rotors_description/urdf/iris_base.xacro (robot description, xacro)
@@ -7,5 +7,4 @@
   <xacro:arg name='mavlink_addr' default='INADDR_ANY' />
   <xacro:arg name='mavlink_udp_port' default='14560' />
-  <xacro:arg name='mavlink_tcp_port' default='4560' />
   <xacro:arg name='serial_enabled' default='false' />
   <xacro:arg name='serial_device' default='/dev/ttyACM0' />
@@ -13,12 +12,6 @@
   <xacro:arg name='qgc_addr' default='INADDR_ANY' />
   <xacro:arg name='qgc_udp_port' default='14550' />
-  <xacro:arg name='sdk_addr' default='INADDR_ANY' />
-  <xacro:arg name='sdk_udp_port' default='14540' />
   <xacro:arg name='hil_mode' default='false' />
   <xacro:arg name='hil_state_level' default='false' />
-  <xacro:arg name='send_vision_estimation' default='false' />
-  <xacro:arg name='send_odometry' default='false' />
-  <xacro:arg name='enable_lockstep' default='true' />
-  <xacro:arg name='use_tcp' default='true' />
   <xacro:arg name='vehicle_is_tailsitter' default='false' />
   <xacro:arg name='visual_material' default='DarkGrey' />
@@ -45,5 +38,5 @@
         />
   </xacro:if>
-  <!-- Instantiate gps plugin. -->
+    <!-- Instantiate gps plugin. -->
   <xacro:gps_plugin_macro
     namespace="${namespace}"
@@ -51,21 +44,4 @@
     >
   </xacro:gps_plugin_macro>
-  <!-- Instantiate magnetometer plugin. -->
-  <xacro:magnetometer_plugin_macro
-    namespace="${namespace}"
-    pub_rate="20"
-    noise_density="0.0004"
-    random_walk="0.0000064"
-    bias_correlation_time="600"
-    mag_topic="/mag"
-    >
-  </xacro:magnetometer_plugin_macro>
-  <!-- Instantiate barometer plugin. -->
-  <xacro:barometer_plugin_macro
-    namespace="${namespace}"
-    pub_rate="10"
-    baro_topic="/baro"
-    >
-  </xacro:barometer_plugin_macro>
   <xacro:if value="$(arg enable_mavlink_interface)">
   <!-- Instantiate mavlink telemetry interface. -->
@@ -74,9 +50,6 @@
     imu_sub_topic="/imu"
     gps_sub_topic="/gps"
-    mag_sub_topic="/mag"
-    baro_sub_topic="/baro"
     mavlink_addr="$(arg mavlink_addr)"
     mavlink_udp_port="$(arg mavlink_udp_port)"
-    mavlink_tcp_port="$(arg mavlink_tcp_port)"
     serial_enabled="$(arg serial_enabled)"
     serial_device="$(arg serial_device)"
@@ -84,13 +57,7 @@
     qgc_addr="$(arg qgc_addr)"
     qgc_udp_port="$(arg qgc_udp_port)"
-    sdk_addr="$(arg sdk_addr)"
-    sdk_udp_port="$(arg sdk_udp_port)"
     hil_mode="$(arg hil_mode)"
     hil_state_level="$(arg hil_state_level)"
     vehicle_is_tailsitter="$(arg vehicle_is_tailsitter)"
-    send_vision_estimation="$(arg send_vision_estimation)"
-    send_odometry="$(arg send_odometry)"
-    enable_lockstep="$(arg enable_lockstep)"
-    use_tcp="$(arg use_tcp)"
     >
   </xacro:mavlink_interface_macro>
